File: sch/mssaPIC12.sch (EAGLE design)
At the start: 30 parts, among them IC1 PIC12F675P, IC2 7805L, Q1 BC550C, Q2 BC550C

Commit message: Add files via upload
Other:
- note added: "or PIC12F683"
Changed lines of the file:
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@@
 <plain>
 <text x="25.4" y="109.22" size="3.81" layer="91">LZ2HV T-Cross</text>
+<text x="63.5" y="30.48" size="1.778" layer="91">or PIC12F683</text>
 </plain>
 <instances>
