File: sch/mssaPIC12.sch (EAGLE design)
At the start: 30 parts, among them IC1 PIC12F675P, IC2 7805L, Q1 BC550C, Q2 BC550C

Commit message: SSA v.034
Parts:
- added D4: 1N4148DO35-7, diode:1N4148DO35-7
- added R9: 100, rcl:R-EU_0204/5
Connections:
- new net N$11: D4.C, R1.2
- new net N$16: PAD3.P, R9.2
- net N$13: now also C9.1; no longer C9.2
- net N$2: now also D4.A; no longer R1.2
- net N$9: now also C9.2, R9.1; no longer C9.1, PAD3.P
Other:
- moved on the sheet: C9, PAD2, PAD3, R1

Commit message: Add files via upload
Parts:
- added R11: 33k, rcl:R-EU_0207/2V
- R1: value 15k -> 10k
- R9: device rcl:R-EU_0204/5 -> rcl:R-EU_0207/2V
Connections:
- net N$13: now also R11.2
- net N$9: now also R11.1
Other:
- moved on the sheet: D2, R9
Changed lines of the file:
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@@
 <part name="Q1" library="transistor-npn" library_urn="urn:adsk.eagle:library:398" deviceset="BC550*" device="" package3d_urn="urn:adsk.eagle:package:28989/2" technology="C"/>
 <part name="GND5" library="supply1" deviceset="GND" device=""/>
-<part name="R1" library="rcl" library_urn="urn:adsk.eagle:library:334" deviceset="R-EU_" device="0207/7" package3d_urn="urn:adsk.eagle:package:23493/2" value="15k"/>
+<part name="R1" library="rcl" library_urn="urn:adsk.eagle:library:334" deviceset="R-EU_" device="0207/7" package3d_urn="urn:adsk.eagle:package:23493/2" value="10k"/>
 <part name="R2" library="rcl" library_urn="urn:adsk.eagle:library:334" deviceset="R-EU_" device="0207/7" package3d_urn="urn:adsk.eagle:package:23493/2" value="15k"/>
 <part name="R3" library="rcl" library_urn="urn:adsk.eagle:library:334" deviceset="R-EU_" device="0207/7" package3d_urn="urn:adsk.eagle:package:23493/2" value="8.2k"/>
@@
 <part name="LED1" library="led" library_urn="urn:adsk.eagle:library:259" deviceset="LED" device="3MM" package3d_urn="urn:adsk.eagle:package:15797/1" value="MAIN"/>
 <part name="GND15" library="supply1" deviceset="GND" device=""/>
-<part name="R9" library="rcl" library_urn="urn:adsk.eagle:library:334" deviceset="R-EU_" device="0204/5" package3d_urn="urn:adsk.eagle:package:23488/1" value="100"/>
+<part name="R9" library="rcl" library_urn="urn:adsk.eagle:library:334" deviceset="R-EU_" device="0207/2V" package3d_urn="urn:adsk.eagle:package:23490/1" value="100"/>
 <part name="D4" library="diode" library_urn="urn:adsk.eagle:library:210" deviceset="1N4148" device="DO35-7" package3d_urn="urn:adsk.eagle:package:43339/2"/>
+<part name="R11" library="rcl" library_urn="urn:adsk.eagle:library:334" deviceset="R-EU_" device="0207/2V" package3d_urn="urn:adsk.eagle:package:23490/1" value="33k"/>
 </parts>
 <sheets>
@@
 <attribute name="VALUE" x="12.7" y="48.26" size="1.778" layer="96"/>
 </instance>
-<instance part="D2" gate="1" x="-5.08" y="71.12" smashed="yes">
-<attribute name="NAME" x="-2.54" y="71.6026" size="1.778" layer="95"/>
-<attribute name="VALUE" x="-2.54" y="68.8086" size="1.778" layer="96"/>
+<instance part="D2" gate="1" x="0" y="71.12" smashed="yes">
+<attribute name="NAME" x="2.54" y="71.6026" size="1.778" layer="95"/>
+<attribute name="VALUE" x="2.54" y="68.8086" size="1.778" layer="96"/>
 </instance>
 <instance part="D3" gate="1" x="-12.7" y="48.26" smashed="yes" rot="R90">
@@
 <attribute name="VALUE" x="48.26" y="22.86" size="1.778" layer="96"/>
 </instance>
-<instance part="R9" gate="G$1" x="-12.7" y="88.9" smashed="yes" rot="R90">
-<attribute name="NAME" x="-14.1986" y="85.09" size="1.778" layer="95" rot="R90"/>
-<attribute name="VALUE" x="-9.398" y="85.09" size="1.778" layer="96" rot="R90"/>
+<instance part="R9" gate="G$1" x="-12.7" y="91.44" smashed="yes" rot="R90">
+<attribute name="NAME" x="-14.1986" y="87.63" size="1.778" layer="95" rot="R90"/>
+<attribute name="VALUE" x="-9.398" y="87.63" size="1.778" layer="96" rot="R90"/>
 </instance>
 <instance part="D4" gate="G$1" x="53.34" y="60.96" smashed="yes" rot="R180">
 <attribute name="NAME" x="50.8" y="60.4774" size="1.778" layer="95" rot="R180"/>
 <attribute name="VALUE" x="58.42" y="65.8114" size="1.778" layer="96" rot="R180"/>
+</instance>
+<instance part="R11" gate="G$1" x="-5.08" y="78.74" smashed="yes" rot="R270">
+<attribute name="NAME" x="-3.5814" y="82.55" size="1.778" layer="95" rot="R270"/>
+<attribute name="VALUE" x="-8.382" y="82.55" size="1.778" layer="96" rot="R270"/>
 </instance>
 </instances>
@@
 <wire x1="15.24" y1="71.12" x2="5.08" y2="71.12" width="0.1524" layer="91"/>
 <pinref part="D2" gate="1" pin="C"/>
-<wire x1="-2.54" y1="71.12" x2="5.08" y2="71.12" width="0.1524" layer="91"/>
+<wire x1="2.54" y1="71.12" x2="5.08" y2="71.12" width="0.1524" layer="91"/>
 <junction x="5.08" y="71.12"/>
 </segment>
@@
 <wire x1="-12.7" y1="50.8" x2="-12.7" y2="71.12" width="0.1524" layer="91"/>
 <pinref part="D2" gate="1" pin="A"/>
-<wire x1="-12.7" y1="71.12" x2="-7.62" y2="71.12" width="0.1524" layer="91"/>
+<wire x1="-12.7" y1="71.12" x2="-5.08" y2="71.12" width="0.1524" layer="91"/>
 <pinref part="C9" gate="G$1" pin="1"/>
+<wire x1="-5.08" y1="71.12" x2="-2.54" y2="71.12" width="0.1524" layer="91"/>
 <wire x1="-12.7" y1="71.12" x2="-12.7" y2="73.66" width="0.1524" layer="91"/>
 <junction x="-12.7" y="71.12"/>
+<pinref part="R11" gate="G$1" pin="2"/>
+<wire x1="-5.08" y1="73.66" x2="-5.08" y2="71.12" width="0.1524" layer="91"/>
+<junction x="-5.08" y="71.12"/>
 </segment>
 </net>
@@
 <pinref part="R9" gate="G$1" pin="1"/>
 <wire x1="-12.7" y1="81.28" x2="-12.7" y2="83.82" width="0.1524" layer="91"/>
+<pinref part="R11" gate="G$1" pin="1"/>
+<wire x1="-12.7" y1="83.82" x2="-12.7" y2="86.36" width="0.1524" layer="91"/>
+<wire x1="-5.08" y1="83.82" x2="-12.7" y2="83.82" width="0.1524" layer="91"/>
+<junction x="-12.7" y="83.82"/>
 </segment>
 </net>
@@
 <pinref part="R9" gate="G$1" pin="2"/>
 <pinref part="PAD3" gate="P" pin="P"/>
-<wire x1="-12.7" y1="93.98" x2="-12.7" y2="96.52" width="0.1524" layer="91"/>
-</segment>
-</net>
+</segment>
+</net>

Commit message: Add files via upload
Parts:
- C7: value 220n -> 470n
Changed lines of the file:
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@@
 <part name="C6" library="capacitor-wima" deviceset="C" device="5/2.5" value="2.2u"/>
 <part name="GND12" library="supply1" deviceset="GND" device=""/>
-<part name="C7" library="capacitor-wima" deviceset="C" device="5/2.5" value="220n"/>
+<part name="C7" library="capacitor-wima" deviceset="C" device="5/2.5" value="470n"/>
 <part name="GND13" library="supply1" deviceset="GND" device=""/>
 <part name="D2" library="diode" library_urn="urn:adsk.eagle:library:210" deviceset="1N4004" device="" package3d_urn="urn:adsk.eagle:package:43336/1"/>
