File: sch/smd/pic12f683_004/mssaPIC12smd.brd (EAGLE design)
At the start: 42 x 30 mm, 45 parts, among them IC2 78L05F, IC3 PIC12F683SN, Q1 BC817, Q2 BC817, Q3 BC807

Commit message: Add files via upload
Parts:
- added R16: 33k, rcl:M1206
- R1: value 15k -> 10k
- R2: value 22k -> 15k
- R8: value 50 -> 100
- moved R8 3.00 mm to (5.90, 7.50)
- moved D3 0.36 mm to (13.4, 8.10)
Connections:
- net N$13: now also R16.2
- net N$2: now also R16.1
Routing:
- net N$13: track 4.86 -> 10.8 mm
- net N$2: track 5.77 -> 9.36 mm
- net GND: track 85.5 -> 85.1 mm, vias 13 -> 14
Changed lines of the file:
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@@
 <attribute name="VALUE" x="19.51" y="8.028" size="1.27" layer="27" ratio="10" display="off"/>
 </element>
-<element name="R1" library="rcl" library_urn="urn:adsk.eagle:library:334" package="M1206" package3d_urn="urn:adsk.eagle:package:23566/2" value="15k" x="28.138" y="12.05" smashed="yes" rot="R270">
+<element name="R1" library="rcl" library_urn="urn:adsk.eagle:library:334" package="M1206" package3d_urn="urn:adsk.eagle:package:23566/2" value="10k" x="28.138" y="12.05" smashed="yes" rot="R270">
 <attribute name="NAME" x="24.862" y="13.698" size="1.27" layer="25" ratio="10"/>
 <attribute name="POPULARITY" value="17" x="28.138" y="12.05" size="1.778" layer="27" rot="R270" display="off"/>
@@
 <attribute name="VALUE" x="25.703" y="12.4106" size="1.27" layer="27" ratio="10" rot="R270"/>
 </element>
-<element name="R2" library="rcl" library_urn="urn:adsk.eagle:library:334" package="M1206" package3d_urn="urn:adsk.eagle:package:23566/2" value="22k" x="26.65" y="3.062" smashed="yes" rot="R180">
+<element name="R2" library="rcl" library_urn="urn:adsk.eagle:library:334" package="M1206" package3d_urn="urn:adsk.eagle:package:23566/2" value="15k" x="26.65" y="3.062" smashed="yes" rot="R180">
 <attribute name="NAME" x="29.098" y="5.638" size="1.27" layer="25" ratio="10" rot="R180"/>
 <attribute name="POPULARITY" value="17" x="26.65" y="3.062" size="1.778" layer="27" rot="R180" display="off"/>
@@
 <attribute name="VALUE" x="25.524" y="5.513" size="1.27" layer="27" rot="R180"/>
 </element>
-<element name="D3" library="diode" library_urn="urn:adsk.eagle:library:210" package="SOD-123_MINI-SMA" package3d_urn="urn:adsk.eagle:package:43457/2" value="1N4001" x="13.1" y="8.3" smashed="yes" rot="R90">
-<attribute name="NAME" x="11.976" y="11.143" size="1.27" layer="25"/>
-<attribute name="POPULARITY" value="0" x="13.1" y="8.3" size="1.778" layer="27" rot="R90" display="off"/>
-<attribute name="VALUE" x="15.513" y="6.776" size="1.27" layer="27" rot="R90"/>
+<element name="D3" library="diode" library_urn="urn:adsk.eagle:library:210" package="SOD-123_MINI-SMA" package3d_urn="urn:adsk.eagle:package:43457/2" value="1N4001" x="13.4" y="8.1" smashed="yes" rot="R90">
+<attribute name="NAME" x="12.276" y="10.943" size="1.27" layer="25"/>
+<attribute name="POPULARITY" value="0" x="13.4" y="8.1" size="1.778" layer="27" rot="R90" display="off"/>
+<attribute name="VALUE" x="15.813" y="6.576" size="1.27" layer="27" rot="R90"/>
 </element>
 <element name="R7" library="rcl" library_urn="urn:adsk.eagle:library:334" package="M1206" package3d_urn="urn:adsk.eagle:package:23566/2" value="15k" x="21.8" y="24.6" smashed="yes" rot="R270">
@@
 <attribute name="VALUE" x="19.26" y="25.87" size="1.27" layer="27" rot="R270"/>
 </element>
-<element name="R8" library="rcl" library_urn="urn:adsk.eagle:library:334" package="M1206" package3d_urn="urn:adsk.eagle:package:23566/2" value="50" x="8.9" y="7.5" smashed="yes" rot="R180">
-<attribute name="NAME" x="5.07" y="8.87" size="1.27" layer="25" rot="R270"/>
-<attribute name="POPULARITY" value="17" x="8.9" y="7.5" size="1.778" layer="27" rot="R180" display="off"/>
-<attribute name="SPICEPREFIX" value="R" x="8.9" y="7.5" size="1.778" layer="27" rot="R180" display="off"/>
-<attribute name="VALUE" x="10.17" y="10.04" size="1.27" layer="27" rot="R180"/>
+<element name="R8" library="rcl" library_urn="urn:adsk.eagle:library:334" package="M1206" package3d_urn="urn:adsk.eagle:package:23566/2" value="100" x="5.9" y="7.5" smashed="yes" rot="R180">
+<attribute name="NAME" x="2.07" y="8.87" size="1.27" layer="25" rot="R270"/>
+<attribute name="POPULARITY" value="17" x="5.9" y="7.5" size="1.778" layer="27" rot="R180" display="off"/>
+<attribute name="SPICEPREFIX" value="R" x="5.9" y="7.5" size="1.778" layer="27" rot="R180" display="off"/>
+<attribute name="VALUE" x="7.17" y="10.04" size="1.27" layer="27" rot="R180"/>
 </element>
 <element name="R9" library="rcl" library_urn="urn:adsk.eagle:library:334" package="R0603" package3d_urn="urn:adsk.eagle:package:23555/3" value="0" x="22" y="11.9" smashed="yes" rot="R270">
@@
 <attribute name="POPULARITY" value="0" x="27.2" y="8.1" size="1.778" layer="27" display="off"/>
 <attribute name="VALUE" x="24.152" y="5.687" size="1.27" layer="27"/>
+</element>
+<element name="R16" library="rcl" library_urn="urn:adsk.eagle:library:334" package="M1206" package3d_urn="urn:adsk.eagle:package:23566/2" value="33k" x="10.4" y="9.3" smashed="yes" rot="R90">
+<attribute name="NAME" x="9.13" y="8.03" size="1.27" layer="25" rot="R90"/>
+<attribute name="POPULARITY" value="17" x="10.4" y="9.3" size="1.778" layer="27" rot="R90" display="off"/>
+<attribute name="SPICEPREFIX" value="R" x="10.4" y="9.3" size="1.778" layer="27" rot="R90" display="off"/>
+<attribute name="VALUE" x="12.94" y="8.03" size="1.27" layer="27" rot="R90"/>
 </element>
 </elements>
@@
 <contactref element="R7" pad="1"/>
 <wire x1="21.8" y1="26" x2="21.8" y2="27.2" width="1.27" layer="1"/>
-<wire x1="14.620125" y1="9.679875" x2="13.520125" y2="9.679875" width="1.27" layer="1"/>
-<wire x1="13.1" y1="10.1" x2="13.520125" y2="9.679875" width="1.27" layer="1"/>
+<wire x1="14.620125" y1="9.679875" x2="13.620125" y2="9.679875" width="1.27" layer="1"/>
+<wire x1="13.4" y1="9.9" x2="13.620125" y2="9.679875" width="1.27" layer="1"/>
 <wire x1="14.8" y1="9.5" x2="16" y2="9.5" width="1.27" layer="1"/>
 <wire x1="16" y1="9.5" x2="16.3" y2="9.5" width="1.27" layer="1"/>
@@
 <wire x1="35.7" y1="1.7" x2="35.992" y2="1.408" width="0.4064" layer="1"/>
 <wire x1="35.992" y1="1.408" x2="35.992" y2="0.508" width="0.4064" layer="1"/>
+<via x="13.7" y="11.7" extent="1-16" drill="0.6096"/>
 </signal>
 <signal name="N$1">
@@
 <contactref element="D2" pad="A"/>
 <contactref element="C11" pad="2"/>
-<wire x1="13.1" y1="6.5" x2="13.1" y2="4.7" width="1.27" layer="1"/>
-<wire x1="13.1" y1="4.7" x2="12.2" y2="3.8" width="1.27" layer="1"/>
+<wire x1="13.4" y1="6.3" x2="13.4" y2="5" width="1.27" layer="1"/>
+<wire x1="13.4" y1="5" x2="12.2" y2="3.8" width="1.27" layer="1"/>
 <wire x1="12.2" y1="3.1" x2="12.2" y2="3.8" width="1.27" layer="1"/>
 <wire x1="12.2" y1="3.1" x2="14.2" y2="3.1" width="1.27" layer="1"/>
+<contactref element="R16" pad="1"/>
+<wire x1="10.4" y1="7.9" x2="12" y2="6.3" width="1.016" layer="1"/>
+<wire x1="12" y1="6.3" x2="13.4" y2="6.3" width="1.016" layer="1"/>
 </signal>
 <signal name="N$13">
 <contactref element="C11" pad="1"/>
 <contactref element="R8" pad="1"/>
-<wire x1="10.3" y1="7.5" x2="9.8" y2="7" width="1.27" layer="1"/>
-<wire x1="9.8" y1="7" x2="9.8" y2="3.7" width="1.27" layer="1"/>
-<wire x1="9.8" y1="3.7" x2="9.2" y2="3.1" width="1.27" layer="1"/>
+<wire x1="9.5" y1="3.1" x2="8.6" y2="4" width="1.27" layer="1"/>
+<wire x1="8.6" y1="5.3" x2="7.3" y2="6.6" width="1.27" layer="1"/>
+<wire x1="7.3" y1="7.5" x2="7.3" y2="6.6" width="1.27" layer="1"/>
+<wire x1="8.6" y1="5.3" x2="8.6" y2="4" width="1.27" layer="1"/>
+<wire x1="9.5" y1="3.1" x2="9.2" y2="3.1" width="1.27" layer="1"/>
+<contactref element="R16" pad="2"/>
+<wire x1="7.3" y1="7.5" x2="7.4" y2="7.6" width="1.016" layer="1"/>
+<wire x1="7.4" y1="8.7" x2="7.4" y2="7.6" width="1.016" layer="1"/>
+<wire x1="7.4" y1="8.7" x2="9.5" y2="10.8" width="1.016" layer="1"/>
+<wire x1="9.5" y1="10.8" x2="10.3" y2="10.8" width="1.016" layer="1"/>
+<wire x1="10.3" y1="10.8" x2="10.4" y2="10.7" width="1.016" layer="1"/>
 </signal>
 <signal name="N$14">
 <contactref element="R8" pad="2"/>
 <contactref element="LED" pad="1"/>
-<wire x1="7.5" y1="7.5" x2="5.72565625" y2="5.72565625" width="1.27" layer="1"/>
-<wire x1="5.6" y1="3.7" x2="5.72565625" y2="5.72565625" width="1.27" layer="1"/>
+<wire x1="4.512090625" y1="3.7" x2="4.5" y2="3.715528125" width="1.27" layer="1"/>
+<wire x1="4.5" y1="7.5" x2="4.5" y2="3.715528125" width="1.27" layer="1"/>
+<wire x1="5.6" y1="3.7" x2="4.512090625" y2="3.7" width="1.27" layer="1"/>
 </signal>
 <signal name="N$15">
